File: FLIPPER_CAN_BUS/FLIPPER_CAN_BUS.kicad_sch (KiCad schematic)
At the start: 21 parts, among them J1 Conn_01x02, J1 Conn_01x08_Socket, J2 Conn_01x10_Socket, U1 TJA1051T/3, U2 MCP2515-xST, U3 AP3602AKTR-G1, Y1 16 Mhz

Commit message: FLIPPER_CAN_BUS
Cambios en diseño
Parts:
- removed R3, R4: 10k, Resistor_SMD:R_0603_1608Metric_Pad0.98x0.95mm_HandSolder, symbol CanBus-rescue:R-Device
- added C10, C11, C9: 0.1uf, Capacitor_SMD:C_0603_1608Metric_Pad1.08x0.95mm_HandSolder, symbol CanBus-rescue:C-Device
- added C12, C14: 10uf, Capacitor_SMD:C_0603_1608Metric_Pad1.08x0.95mm_HandSolder, symbol CanBus-rescue:C-Device
Connections:
- net +3V3: now also C10.1, C12.1
- net +5V: now also C11.1, C14.1, C9.1; no longer J1.1 (Pin_1)
- net GND: now also C10.2, C11.2, C12.2, C14.2, C9.2
- net INT: now also J2.2 (Pin_2)
- net RST: now also J1.7 (Pin_7)
- no-connect marks 15 -> 14
Other:
- note added: "BOOST CONVERTER"
- note added: "MCP2515"
- note added: "PINOUT"
- moved on the sheet: C5, C7, C8, J1, J2, U3

Commit message: got ignore update
Parts:
- removed C6: 47pf, Capacitor_SMD:C_0603_1608Metric_Pad1.08x0.95mm_HandSolder, symbol CanBus-rescue:C-Device
- added C2: 0.1uf, Capacitor_SMD:C_0603_1608Metric_Pad1.08x0.95mm_HandSolder, symbol CanBus-rescue:C-Device
- C1: value .1uf -> 47pf; #LCSC C387984 -> (none); #Manf 0603F104Z160CT -> (none); Manufactura LCSC -> Mouser; manf# (none) -> C0603C470J4GACAUTO
- C10: renamed from C12; #Manf 06035A220JAT4A -> (none); manf# (none) -> 0805YC106KAT2A
- C11: #Manf 06035A220JAT4A -> (none); manf# (none) -> 0603F104Z160CT
- C12: renamed from C8; #Manf 06035A220JAT4A -> (none); manf# (none) -> 0805YC106KAT2A
- C13: renamed from C7; #Manf 06035A220JAT4A -> (none); manf# (none) -> 0805YC106KAT2A
- C3, C4: #Manf 06035A220JAT4A -> (none); manf# (none) -> 0805YA220JAT2A
- C5: renamed from C2; #Manf 06035A220JAT4A -> (none); manf# (none) -> C0603C470J4GACAUTO
- C6: renamed from C5; #Manf 06035A220JAT4A -> (none); manf# (none) -> 0402YD105KAT4A
- C7: renamed from C9; #Manf 06035A220JAT4A -> (none); manf# (none) -> 0603F104Z160CT
- C8: renamed from C14; #Manf 06035A220JAT4A -> (none); manf# (none) -> 0805YC106KAT2A
- C9: renamed from C10; #Manf 06035A220JAT4A -> (none); manf# (none) -> 0603F104Z160CT
- D1: renamed from D2; Manufactura (none) -> Mouser; PROD_ID DIO-12501 -> (none); manf# (none) -> PESD1CAN-UX
- J1, J2: Manufactura (none) -> LCSC
- J1: #Manf --- -> (none); manf# (none) -> ---
- R1: #Manf CRCW080510K0FKEAC -> (none); manf# (none) -> CRCW080510K0FKEAC
- R2: #Manf CRCW080510K0FKEAC -> (none); manf# (none) -> CRCW0805120RFKEAC
- R3: renamed from R5; #Manf CRCW080510K0FKEAC -> (none); manf# (none) -> CRCW080510K0FKEAC
- U1: Manufactura (none) -> Mouser; manf# (none) -> TJA1051T/3,118
- U2: #LCSC C15193 -> (none); #Manf MCP2515-I/ST -> (none); LCSC# (none) -> C15193; Manufactura LCSC -> Mouser; manf# (none) -> MCP2515-I/ST
- U3: Manufactura (none) -> Mouser; manf# (none) -> AP3602AKTR-G1
- Y1: #LCSC C254270 -> (none); #Manf X2C016000B91H-R -> (none); LCSC# (none) -> C254270; manf# (none) -> X2C016000B91H-R
Connections:
- net +3V3: now also C2.2; no longer C1.1
- net CAN_H+: now also C1.1
- net GND: now also C3.1, C4.1, C2.1; no longer C3.2, C4.2, J2.10 (Pin_10), J2.3 (Pin_3)
- net at U2.9 (OSC1), Y1.3: now also C4.2; no longer C4.1
- net at U2.8 (OSC2), Y1.1: now also C3.2; no longer C3.1

Commit message: Correcion
update
Connections:
- net GND: now also J2.10 (Pin_10), J2.3 (Pin_3)
Other:
- note added: "CAN_BUS OUTPUTS"

Commit message: upd PCB
Correcion estetica
Connections:
- net CAN_H+ renamed CAN_H
Other:
- moved on the sheet: C10, C11, C9, R1
