File: FLIPPER_CAN_BUS/FLIPPER_CAN_BUS.kicad_sch (KiCad schematic)
At the start: 24 parts, among them J1 Conn_01x02, J1 Conn_01x08_Socket, J2 Conn_01x10_Socket, U1 TJA1051T/3, U2 MCP2515-xST, U3 AP3602AKTR-G1, Y1 16 Mhz

Commit message: upd
Parts:
- U2: Manufactura Mouser -> Mouser o LCSC
Changed lines of the file:
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@@
       (effects (font (size 1.27 1.27)) hide)
     )
-    (property "Manufactura" "Mouser" (at 64.135 46.228 0)
+    (property "Manufactura" "Mouser o LCSC" (at 64.135 46.228 0)
       (effects (font (size 1.27 1.27)) hide)
     )
@@
   )
   (symbol (lib_id "TJA1051T_3:TJA1051T{slash}3") (at 152.527 41.148 0) (unit 1)
-    (in_bom yes) (on_board yes) (dnp no) (fields_autoplaced)
+    (in_bom yes) (on_board yes) (dnp no)
     (property "Reference" "U1" (at 154.3559 29.21 0)
       (effects (font (size 1.27 1.27)) (justify left))
     )
-    (property "Value" "TJA1051T/3" (at 154.3559 31.75 0)
+    (property "Value" "TJA1051T/3" (at 139.7 30.48 0)
       (effects (font (size 1.27 1.27)) (justify left))
     )

Commit message: upd
CSV
Parts:
- C1, C10, C11, C12, C13, C2, C3, C4, C5, C6, C7, C8, C9, D1, R1, R2, R3, U1, U3: Manufactura Mouser -> (none); Proveedor (none) -> Mouser
- J1, J2: Manufactura LCSC -> (none); manf# PZ2.54-1*20-WZ -> (none)
- J1: Manufactura Steren -> (none); Proveedor (none) -> Steren
- U2: Manufactura Mouser o LCSC -> (none); Proveedor (none) -> LCSC
- Y1: Manufactura LCSC -> (none); Proveedor (none) -> LCSC
Changed lines of the file:
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@@
       (effects (font (size 1.27 1.27)) hide)
     )
-    (property "Manufactura" "Mouser" (at 208.153 106.172 0)
+    (property "Proveedor" "Mouser" (at 208.153 106.172 0)
       (effects (font (size 1.27 1.27)) hide)
     )
@@
       (effects (font (size 1.27 1.27)) hide)
     )
-    (property "Manufactura" "Mouser" (at 205.105 56.134 0)
+    (property "Proveedor" "Mouser" (at 205.105 56.134 0)
       (effects (font (size 1.27 1.27)) hide)
     )
@@
       (effects (font (size 1.27 1.27)) hide)
     )
-    (property "Manufactura" "Mouser" (at 146.558 109.22 0)
+    (property "Proveedor" "Mouser" (at 146.558 109.22 0)
       (effects (font (size 1.27 1.27)) hide)
     )
@@
       (effects (font (size 1.27 1.27)) hide)
     )
-    (property "Manufactura" "Mouser" (at 130.81 49.403 0)
+    (property "Proveedor" "Mouser" (at 130.81 49.403 0)
       (effects (font (size 1.27 1.27)) hide)
     )
@@
       (effects (font (size 1.27 1.27)) hide)
     )
-    (property "Manufactura" "LCSC" (at 29.845 52.324 0)
+    (property "Proveedor" "LCSC" (at 29.845 52.324 0)
       (effects (font (size 1.27 1.27)) hide)
     )
@@
       (effects (font (size 1.27 1.27)) hide)
     )
-    (property "Manufactura" "Mouser" (at 132.334 100.457 0)
+    (property "Proveedor" "Mouser" (at 132.334 100.457 0)
       (effects (font (size 1.27 1.27)) hide)
     )
@@
       (effects (font (size 1.27 1.27)) hide)
     )
-    (property "Manufactura" "Mouser" (at 124.714 100.457 0)
+    (property "Proveedor" "Mouser" (at 124.714 100.457 0)
       (effects (font (size 1.27 1.27)) hide)
     )
@@
       (effects (font (size 1.27 1.27)) hide)
     )
-    (property "Manufactura" "Mouser" (at 220.726 38.608 0)
+    (property "Proveedor" "Mouser" (at 220.726 38.608 0)
       (effects (font (size 1.27 1.27)) hide)
     )
@@
       (effects (font (size 1.27 1.27)) hide)
     )
-    (property "Manufactura" "Mouser" (at 201.295 101.219 0)
+    (property "Proveedor" "Mouser" (at 201.295 101.219 0)
       (effects (font (size 1.27 1.27)) hide)
     )
@@
       (effects (font (size 1.27 1.27)) hide)
     )
-    (property "Manufactura" "Mouser" (at 19.685 48.514 0)
+    (property "Proveedor" "Mouser" (at 19.685 48.514 0)
       (effects (font (size 1.27 1.27)) hide)
     )
@@
       (effects (font (size 1.27 1.27)) hide)
     )
-    (property "Manufactura" "Mouser" (at 19.685 56.134 0)
+    (property "Proveedor" "Mouser" (at 19.685 56.134 0)
       (effects (font (size 1.27 1.27)) hide)
     )
@@
       (effects (font (size 1.27 1.27)) hide)
     )
-    (property "Manufactura" "Mouser" (at 225.933 100.457 0)
+    (property "Proveedor" "Mouser" (at 225.933 100.457 0)
       (effects (font (size 1.27 1.27)) hide)
     )
@@
       (effects (font (size 1.27 1.27)) hide)
     )
-    (property "LCSC Part Number" "" (at 80.645 103.886 0)
-      (effects (font (size 1.27 1.27)) hide)
-    )
-    (property "LCSC Price/Stock" "" (at 80.645 103.886 0)
-      (effects (font (size 1.27 1.27)) hide)
-    )
     (property "LCSC#" "C5360907" (at 80.645 103.886 0)
       (effects (font (size 1.27 1.27)) hide)
@@
       (effects (font (size 1.27 1.27)) hide)
     )
-    (property "manf#" "PZ2.54-1*20-WZ" (at 80.645 103.886 0)
-      (effects (font (size 1.27 1.27)) hide)
-    )
-    (property "Manufactura" "LCSC" (at 80.645 103.886 0)
+    (property "manf#" "" (at 80.645 103.886 0)
       (effects (font (size 1.27 1.27)) hide)
     )
@@
       (effects (font (size 1.27 1.27)) hide)
     )
-    (property "manf#" "PZ2.54-1*20-WZ" (at 50.165 101.473 0)
-      (effects (font (size 1.27 1.27)) hide)
-    )
-    (property "Manufactura" "LCSC" (at 50.165 101.473 0)
+    (property "manf#" "" (at 50.165 101.473 0)
       (effects (font (size 1.27 1.27)) hide)
     )
@@
       (effects (font (size 1.27 1.27)) hide)
     )
-    (property "Manufactura" "Mouser" (at 155.194 97.282 0)
+    (property "Proveedor" "Mouser" (at 155.194 97.282 0)
       (effects (font (size 1.27 1.27)) hide)
     )
@@
       (effects (font (size 1.27 1.27)) hide)
     )
-    (property "Manufactura" "Mouser" (at 204.724 21.082 0)
+    (property "Proveedor" "Mouser" (at 204.724 21.082 0)
       (effects (font (size 1.27 1.27)) hide)
     )
@@
       (effects (font (size 1.27 1.27)) hide)
     )
-    (property "Manufactura" "Mouser" (at 235.839 33.528 0)
+    (property "Proveedor" "Mouser" (at 235.839 33.528 0)
       (effects (font (size 1.27 1.27)) hide)
     )
@@
       (effects (font (size 1.27 1.27)) hide)
     )
-    (property "Manufactura" "Mouser" (at 58.039 23.368 0)
+    (property "Proveedor" "Mouser" (at 58.039 23.368 0)
       (effects (font (size 1.27 1.27)) hide)
     )
@@
       (effects (font (size 1.27 1.27)) hide)
     )
-    (property "Manufactura" "Mouser" (at 35.687 29.845 0)
+    (property "Proveedor" "Mouser" (at 35.687 29.845 0)
       (effects (font (size 1.27 1.27)) hide)
     )
@@
       (effects (font (size 1.27 1.27)) hide)
     )
-    (property "Manufactura" "Mouser o LCSC" (at 64.135 46.228 0)
+    (property "Proveedor" "LCSC" (at 64.135 46.228 0)
       (effects (font (size 1.27 1.27)) hide)
     )
@@
       (effects (font (size 1.27 1.27)) hide)
     )
-    (property "Manufactura" "Steren " (at 276.352 37.084 0)
+    (property "Proveedor" "Steren" (at 276.352 37.084 0)
       (effects (font (size 1.27 1.27)) hide)
     )
@@
       (effects (font (size 1.27 1.27)) hide)
     )
-    (property "Manufactura" "Mouser" (at 218.313 100.457 0)
+    (property "Proveedor" "Mouser" (at 218.313 100.457 0)
       (effects (font (size 1.27 1.27)) hide)
     )
@@
       (effects (font (size 1.27 1.27)) hide)
     )
-    (property "Manufactura" "Mouser" (at 152.527 41.148 0)
+    (property "Proveedor" "Mouser" (at 152.527 41.148 0)
       (effects (font (size 1.27 1.27)) hide)
     )
@@
       (effects (font (size 1.27 1.27)) hide)
     )
-    (property "Manufactura" "Mouser" (at 240.284 100.584 0)
-      (effects (font (size 1.27 1.27)) hide)
-    )
+    (property "Proveedor" "Mouser" (at 240.284 100.584 0)
+      (effects (font (size 1.27 1.27)) hide)
+    )

Commit message: upd
upd bom
Parts:
- C10, C12, C13, C8: manf# 0805YC106KAT2A -> KAM15CT70J106KT
- C3, C4: manf# 0805YA220JAT2A -> 06035A220JAT2A
- C6: manf# 0402YD105KAT4A -> 06035C105KAT2A
- D1: footprint SOT23-3 -> Package_TO_SOT_SMD:SOT-323_SC-70
- J1, J2: LCSC# C5360907 -> (none); Proveedor LCSC -> Mouser; manf# (none) -> M20-9961045
- R1, R3: manf# CRCW080510K0FKEAC -> RP0603DRD0710KL
- R2: manf# CRCW0805120RFKEAC -> CRGH0603J120R
- U1: footprint SOT96-1 -> Package_SO:SOIC-8_3.9x4.9mm_P1.27mm
- U2: manf# MCP2515-I/ST -> (none)
- U3: footprint footprints:SOT-23-6_DIO -> Package_TO_SOT_SMD:TSOT-23-6
- Y1: manf# X2C016000B91H-R -> (none)
Changed lines of the file:
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@@
       (effects (font (size 1.27 1.27)) hide)
     )
-    (property "Datasheet" "https://www.mouser.mx/datasheet/2/40/AVX_X7RDielectric_777024-1853642.pdf" (at 208.153 106.172 0)
-      (effects (font (size 1.27 1.27)) hide)
-    )
-    (property "manf#" "0805YC106KAT2A" (at 208.153 106.172 0)
+    (property "Datasheet" "https://www.mouser.mx/datasheet/2/40/KYOCERA_AutoMLCCKAM-3106308.pdf" (at 208.153 106.172 0)
+      (effects (font (size 1.27 1.27)) hide)
+    )
+    (property "manf#" "KAM15CT70J106KT" (at 208.153 106.172 0)
       (effects (font (size 1.27 1.27)) hide)
     )
@@
       (effects (font (size 1.27 1.27)) hide)
     )
-    (property "Datasheet" "https://www.mouser.mx/datasheet/2/40/AVX_X7RDielectric_777024-1853642.pdf" (at 146.558 109.22 0)
-      (effects (font (size 1.27 1.27)) hide)
-    )
-    (property "manf#" "0805YC106KAT2A" (at 146.558 109.22 0)
+    (property "Datasheet" "https://www.mouser.mx/datasheet/2/40/KYOCERA_AutoMLCCKAM-3106308.pdf" (at 146.558 109.22 0)
+      (effects (font (size 1.27 1.27)) hide)
+    )
+    (property "manf#" "KAM15CT70J106KT" (at 146.558 109.22 0)
       (effects (font (size 1.27 1.27)) hide)
     )
@@
       (effects (font (size 1.27 1.27)) hide)
     )
-    (property "Datasheet" "https://www.mouser.mx/datasheet/2/427/crcwce3-1762584.pdf" (at 130.81 49.403 0)
-      (effects (font (size 1.27 1.27)) hide)
-    )
-    (property "manf#" "CRCW080510K0FKEAC" (at 130.81 49.403 0)
+    (property "Datasheet" "https://www.mouser.mx/datasheet/2/447/PYu_RP_51_RoHS_L_0-3071169.pdf" (at 130.81 49.403 0)
+      (effects (font (size 1.27 1.27)) hide)
+    )
+    (property "manf#" "RP0603DRD0710KL" (at 130.81 49.403 0)
       (effects (font (size 1.27 1.27)) hide)
     )
@@
       (effects (font (size 1.27 1.27)) hide)
     )
-    (property "manf#" "	X2C016000B91H-R" (at 29.845 52.324 90)
+    (property "manf#" "" (at 29.845 52.324 90)
       (effects (font (size 1.27 1.27)) hide)
     )
@@
       (effects (font (size 1.27 1.27)) hide)
     )
-    (property "Datasheet" "https://www.mouser.mx/datasheet/2/40/AVX_X7RDielectric_777024-1853642.pdf" (at 132.334 100.457 0)
-      (effects (font (size 1.27 1.27)) hide)
-    )
-    (property "manf#" "0805YC106KAT2A" (at 132.334 100.457 0)
+    (property "Datasheet" "https://www.mouser.mx/datasheet/2/40/KYOCERA_AutoMLCCKAM-3106308.pdf" (at 132.334 100.457 0)
+      (effects (font (size 1.27 1.27)) hide)
+    )
+    (property "manf#" "KAM15CT70J106KT" (at 132.334 100.457 0)
       (effects (font (size 1.27 1.27)) hide)
     )
@@
       (effects (font (size 1.27 1.27)) hide)
     )
-    (property "Datasheet" "https://www.mouser.mx/datasheet/2/427/crcwce3-1762584.pdf" (at 220.726 38.608 0)
-      (effects (font (size 1.27 1.27)) hide)
-    )
-    (property "manf#" "CRCW0805120RFKEAC" (at 220.726 38.608 0)
+    (property "Datasheet" "https://www.mouser.mx/datasheet/2/418/5/ENG_DS_1773204_1_F-717776.pdf" (at 220.726 38.608 0)
+      (effects (font (size 1.27 1.27)) hide)
+    )
+    (property "manf#" "CRGH0603J120R" (at 220.726 38.608 0)
       (effects (font (size 1.27 1.27)) hide)
     )
@@
       (effects (font (size 1.524 1.524)))
     )
-    (property "Footprint" "footprints:SOT-23-6_DIO" (at 201.295 101.219 0)
+    (property "Footprint" "Package_TO_SOT_SMD:TSOT-23-6" (at 201.295 101.219 0)
       (effects (font (size 1.27 1.27) italic) hide)
     )
@@
       (effects (font (size 1.27 1.27)) hide)
     )
-    (property "Datasheet" "https://www.mouser.mx/datasheet/2/40/C0GNP0_Dielectric-951274.pdf" (at 19.685 48.514 0)
-      (effects (font (size 1.27 1.27)) hide)
-    )
-    (property "manf#" "0805YA220JAT2A" (at 19.685 48.514 0)
+    (property "Datasheet" " https://www.mouser.mx/datasheet/2/40/C0GNP0_Dielectric-951274.pdf" (at 19.685 48.514 0)
+      (effects (font (size 1.27 1.27)) hide)
+    )
+    (property "manf#" "06035A220JAT2A" (at 19.685 48.514 0)
       (effects (font (size 1.27 1.27)) hide)
     )
@@
       (effects (font (size 1.27 1.27)) hide)
     )
-    (property "Datasheet" "https://www.mouser.mx/datasheet/2/40/C0GNP0_Dielectric-951274.pdf" (at 19.685 56.134 0)
-      (effects (font (size 1.27 1.27)) hide)
-    )
-    (property "manf#" "0805YA220JAT2A" (at 19.685 56.134 0)
+    (property "Datasheet" " https://www.mouser.mx/datasheet/2/40/C0GNP0_Dielectric-951274.pdf" (at 19.685 56.134 0)
+      (effects (font (size 1.27 1.27)) hide)
+    )
+    (property "manf#" "06035A220JAT2A" (at 19.685 56.134 0)
       (effects (font (size 1.27 1.27)) hide)
     )
@@
       (effects (font (size 1.27 1.27)) hide)
     )
-    (property "Datasheet" "https://www.mouser.mx/datasheet/2/40/AVX_X7RDielectric_777024-1853642.pdf" (at 225.933 100.457 0)
-      (effects (font (size 1.27 1.27)) hide)
-    )
-    (property "manf#" "0805YC106KAT2A" (at 225.933 100.457 0)
+    (property "Datasheet" "https://www.mouser.mx/datasheet/2/40/KYOCERA_AutoMLCCKAM-3106308.pdf" (at 225.933 100.457 0)
+      (effects (font (size 1.27 1.27)) hide)
+    )
+    (property "manf#" "KAM15CT70J106KT" (at 225.933 100.457 0)
       (effects (font (size 1.27 1.27)) hide)
     )
@@
       (effects (font (size 1.27 1.27)) hide)
     )
-    (property "LCSC#" "C5360907" (at 80.645 103.886 0)
-      (effects (font (size 1.27 1.27)) hide)
-    )
-    (property "Proveedor" "LCSC" (at 80.645 103.886 0)
-      (effects (font (size 1.27 1.27)) hide)
-    )
-    (property "manf#" "" (at 80.645 103.886 0)
+    (property "Proveedor" "Mouser" (at 80.645 103.886 0)
+      (effects (font (size 1.27 1.27)) hide)
+    )
+    (property "manf#" "M20-9961045" (at 80.645 103.886 0)
       (effects (font (size 1.27 1.27)) hide)
     )
@@
       (effects (font (size 1.27 1.27)) hide)
     )
-    (property "LCSC#" "C5360907" (at 50.165 101.473 0)
-      (effects (font (size 1.27 1.27)) hide)
-    )
-    (property "Proveedor" "LCSC" (at 50.165 101.473 0)
-      (effects (font (size 1.27 1.27)) hide)
-    )
-    (property "manf#" "" (at 50.165 101.473 0)
+    (property "LCSC#" "" (at 50.165 101.473 0)
+      (effects (font (size 1.27 1.27)) hide)
+    )
+    (property "Proveedor" "Mouser" (at 50.165 101.473 0)
+      (effects (font (size 1.27 1.27)) hide)
+    )
+    (property "manf#" "M20-9961045" (at 50.165 101.473 0)
       (effects (font (size 1.27 1.27)) hide)
     )
@@
       (effects (font (size 1.27 1.27)) hide)
     )
-    (property "Datasheet" "https://www.mouser.mx/datasheet/2/40/AVX_cx5r_776519-1853698.pdf" (at 155.194 97.282 0)
-      (effects (font (size 1.27 1.27)) hide)
-    )
-    (property "manf#" "0402YD105KAT4A" (at 155.194 97.282 0)
+    (property "Datasheet" "https://www.mouser.mx/datasheet/2/40/AVX_X7RDielectric_777024-1853642.pdf" (at 155.194 97.282 0)
+      (effects (font (size 1.27 1.27)) hide)
+    )
+    (property "manf#" "06035C105KAT2A" (at 155.194 97.282 0)
       (effects (font (size 1.27 1.27)) hide)
     )
@@
       (effects (font (size 1.27 1.27)))
     )
-    (property "Footprint" "SOT23-3" (at 235.839 33.528 0)
+    (property "Footprint" "Package_TO_SOT_SMD:SOT-323_SC-70" (at 235.839 33.528 0)
       (effects (font (size 1.27 1.27)) (justify bottom) hide)
     )
@@
       (effects (font (size 1.27 1.27)) hide)
     )
-    (property "Datasheet" "https://www.mouser.mx/datasheet/2/427/crcwce3-1762584.pdf" (at 35.687 29.845 0)
-      (effects (font (size 1.27 1.27)) hide)
-    )
-    (property "manf#" "CRCW080510K0FKEAC" (at 35.687 29.845 0)
+    (property "Datasheet" "https://www.mouser.mx/datasheet/2/447/PYu_RP_51_RoHS_L_0-3071169.pdf" (at 35.687 29.845 0)
+      (effects (font (size 1.27 1.27)) hide)
+    )
+    (property "manf#" "RP0603DRD0710KL" (at 35.687 29.845 0)
       (effects (font (size 1.27 1.27)) hide)
     )
@@
       (effects (font (size 1.27 1.27)) hide)
     )
-    (property "manf#" "MCP2515-I/ST" (at 64.135 46.228 0)
+    (property "manf#" "" (at 64.135 46.228 0)
       (effects (font (size 1.27 1.27)) hide)
     )
@@
       (effects (font (size 1.27 1.27)) (justify left))
     )
-    (property "Footprint" "SOT96-1" (at 152.527 41.148 0)
+    (property "Footprint" "Package_SO:SOIC-8_3.9x4.9mm_P1.27mm" (at 152.527 41.148 0)
       (effects (font (size 1.27 1.27)) (justify bottom) hide)
     )
