File: mags/mags.kicad_pcb (KiCad board)
At the start: 2 copper layers, 66 x 30.7 mm, 4 parts, among them J1 Coil, U1 TC4424, U3 FlipperZero, U4 FlipperZero

Commit message: Fix Flipper_Magspoof
Parts:
- removed U3: FlipperZero, Connector_PinHeader_2.54mm:PinHeader_1x08_P2.54mm_Horizontal
- removed U4: FlipperZero, Connector_PinHeader_2.54mm:PinHeader_1x10_P2.54mm_Horizontal
- added G***: LOGO, Aesthetics:electronic_cats_logo_8x6, F.Cu at (206.3, 61.2)
- added J2: Conn_01x10_Socket, Connector_PinHeader_2.54mm:PinHeader_1x10_P2.54mm_Horizontal, F.Cu at (258.5, 82.5)
- added J3: Conn_01x08_Socket, Connector_PinHeader_2.54mm:PinHeader_1x08_P2.54mm_Horizontal, F.Cu at (217.8, 82.5)
- moved U1 98.3 mm to (226.9, 66.4)
- moved J1 97.6 mm to (237.4, 65.3)
Connections:
- U1 pad 6: /5V -> +5V
Routing:
- net /5V: track 56.5 -> 0.00 mm
- net +5V: track 0.00 -> 55.1 mm
- net /IN_A: track 40.8 -> 35.5 mm
- net /IN_B: track 34.6 -> 30.7 mm
- net /Out_A: track 9.20 -> 8.18 mm
- net /Out_B: track 13.0 -> 13.6 mm
- net GND: vias 1 -> 0
Other:
- board size 66 x 30.7 mm -> 67 x 34 mm
- board text added: "Flipper Zero Magspoof"
- board text removed: "1 2 3 4 5 6 7 8"
- board text removed: "10 11 12 13 14 15 16 17 18"
- board text removed: "9"
