File: mags/mags.kicad_sch (KiCad schematic)
At the start: 4 parts, among them J3 Coil, U3 FlipperZero, U3 TC4424, U4 FlipperZero

Commit message: Fix Flipper_Magspoof
Parts:
- removed U3: FlipperZero, Connector_PinHeader_2.54mm:PinHeader_1x08_P2.54mm_Horizontal, symbol flipper-zen-rescue:FlipperZero-lomalkin_kicad_symbols
- removed U4: FlipperZero, Connector_PinHeader_2.54mm:PinHeader_1x10_P2.54mm_Horizontal, symbol flipper-zen-rescue:FlipperZero-lomalkin_kicad_symbols
- added J2: Conn_01x10_Socket, Connector_PinHeader_2.54mm:PinHeader_1x10_P2.54mm_Horizontal, symbol Connector:Conn_01x10_Socket
- added J3: Conn_01x08_Socket, Connector_PinHeader_2.54mm:PinHeader_1x08_P2.54mm_Horizontal, symbol Connector:Conn_01x08_Socket
Connections:
- net GND: now also J2.1 (Pin_10), J2.8 (Pin_3), J3.1 (Pin_8)
- net IN_A: now also J3.6 (Pin_3)
- net IN_B: now also J3.5 (Pin_4)
- net 5V renamed +5V
- net +5V: now also J3.8 (Pin_1)
- no-connect marks 15 -> 14
Other:
- note added: "+5V"
- note added: "3.3V"
- note added: "GND"
- note added: "PA13"
- note added: "PA14"
- note added: "PA4"
- note added: "PA6"
- note added: "PA7"
- note added: "PB14"
- note added: "PB2"
- note added: "PB3"
- note added: "PB6"
- note added: "PB7"
- note added: "PC0"
- note added: "PC1"
- note added: "PC3"
- note added: "PINOUT DEL FLIPPERO ZERO"
- note added: "TC4424"
- moved on the sheet: J3, U3
