File: MARAUDER_SPOOF/marauder_spoof.kicad_sch (KiCad schematic)
At the start: 26 parts, among them J2 Conn_01x10_Socket, J2 GPS, J3 Coil, J3 Conn_01x08_Socket, J4 Coil, P1 USB_C_Plug_USB2.0, Q1 DMP2004TK-7, Q2 DMP2004TK-7, SW7 RESET, SW8 GPIO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

Commit message: feat(hw): Update Version
Parts:
- renumbered C2 to C1, C3 to C2, C4 to C3, J3 to J1, J2 to J6, R12 to R1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
