File: Marauder/Marauder.kicad_pcb (KiCad board)
At the start: 2 copper layers, 67 x 28 mm, 43 parts, among them J1 Conn_01x08_Socket, J2 Conn_01x08_Socket, J3 Conn_01x10_Socket, J4 GPS, J5 Conn_01x10_Socket, P1 USB_C_Plug_USB2.0, Q1 DMP2004TK-7, Q2 DMP2004TK-7, SW1 RESET, SW2 BOOT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

Commit message: Routing finished of flipper marauder
Parts:
- added kibuzzard-64E4E5CE: G***, kibuzzard-64E4E5CE, B.Cu at (118.6, 88.0)
- added kibuzzard-64E4E792: G***, kibuzzard-64E4E792, B.Cu at (166.5, 73.6)
- added kibuzzard-64E4E7AD: G***, kibuzzard-64E4E7AD, B.Cu at (177.8, 70.3)
- added kibuzzard-64E4E7B8: G***, kibuzzard-64E4E7B8, B.Cu at (171.7, 73.6)
- added kibuzzard-64E4E7C3: G***, kibuzzard-64E4E7C3, B.Cu at (169.1, 73.6)
- added kibuzzard-64E4E837: G***, kibuzzard-64E4E837, F.Cu at (130.4, 69.2)
- added kibuzzard-64E4E889: G***, kibuzzard-64E4E889, F.Cu at (130.3, 82.8)
- kibuzzard-6488EEAF (x3), kibuzzard-6488F75A, kibuzzard-648B91CB, kibuzzard-648B91E6, kibuzzard-648B91FC, kibuzzard-648B921B, kibuzzard-648B922F, kibuzzard-648B923F, kibuzzard-648B93B1, kibuzzard-648B93BF, kibuzzard-648B93D2, kibuzzard-648B93E0, kibuzzard-648B93EF, kibuzzard-648B9401, kibuzzard-648B9410: moved to B.Cu
- moved J4 4.00 mm to (174.2, 70.3)
- moved kibuzzard-6488F75A 3.27 mm to (154.2, 88.0)
- moved kibuzzard-648B91E6 3.26 mm to (128.7, 88.0)
- moved kibuzzard-648B91CB 3.26 mm to (126.2, 88.0)
- moved kibuzzard-648B91FC 3.26 mm to (131.3, 88.0)
- moved kibuzzard-648B921B 3.25 mm to (133.8, 88.0)
- moved kibuzzard-648B923F 3.25 mm to (123.6, 88.0)
- moved kibuzzard-648B922F 3.24 mm to (121.1, 88.0)
- moved kibuzzard-648B9410 3.24 mm to (174.4, 88.0)
- moved kibuzzard-648B93B1 3.23 mm to (156.7, 88.0)
- moved kibuzzard-648B93BF 3.23 mm to (161.8, 88.0)
- moved kibuzzard-6488EEAF 3.15 mm to (136.3, 88.0)
- moved kibuzzard-648B9401 2.92 mm to (171.9, 88.0)
- moved kibuzzard-648B93EF 2.92 mm to (169.4, 88.0)
- moved kibuzzard-648B93E0 2.91 mm to (164.3, 88.0)
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Routing:
- net /LPUART_RX: track 13.8 -> 59.9 mm, vias 0 -> 1
- net /SWCLK: track 0.01 -> 38.8 mm, vias 0 -> 2
- net /SWDIO: track 0.01 -> 34.2 mm, vias 0 -> 2
- net /LPUART_TX: track 19.0 -> 51.7 mm, vias 0 -> 1
- net Net-(Q1-G): track 3.83 -> 15.3 mm
- net +3V3: track 103.7 -> 110.8 mm, vias 6 -> 7
- net /RX: track 53.0 -> 49.3 mm
- net /PB14: track 0.01 -> 3.63 mm
- net /PC3: track 0.02 -> 3.62 mm
- net /PB3: track 0.01 -> 3.61 mm
- net /PB2: track 0.01 -> 3.61 mm
- net /PA7: track 0.00 -> 3.60 mm
- net /PA6: track 0.01 -> 3.61 mm
- net /PA4: track 0.01 -> 3.61 mm
- net +5V: track 0.00 -> 3.60 mm
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- added copper zone on B.Cu, net +3V3
- added copper zone on F.Cu, net +3V3
- added copper zone on B.Cu, net GND
- added copper zone on F.Cu, net GND
- removed copper zone on B.Cu, net (none)
- removed copper zone on F.Cu, net (none)
Other:
- board text added: "Flipper Add-On Marauder v1.1"
- board text removed: "Flipper Add-On Marauder Spoof v1.0"
