File: Marauder/Marauder.kicad_pcb (KiCad board)
At the start: 2 copper layers, 67 x 28 mm, 50 parts, among them J1 Conn_01x08_Socket, J2 Conn_01x08_Socket, J3 Conn_01x10_Socket, J4 GPS, J5 Conn_01x10_Socket, P1 USB_C_Plug_USB2.0, Q1 DMP2004TK-7, Q2 DMP2004TK-7, SW1 RESET, SW2 BOOT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

Commit message: add silkscreen v1.1 to bottom view of flipper marauder
Parts:
- moved G*** 1.92 mm to (160.1, 75.8)
Changed lines of the file:
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@@
   )
   (footprint "Aesthetics:electronic_cats_logo_4x3" (layer "B.Cu")
-    (at 159.76 77.68 180)
+    (at 160.070782 75.782253 180)
     (attr through_hole)
     (fp_text reference "G***" (at 0 0) (layer "B.SilkS") hide
@@
   (gr_line (start 114.51 94.43) (end 114.508414 70.43)
     (stroke (width 0.1) (type default)) (layer "Edge.Cuts"))
+  (gr_text "Flipper Add-On\nMarauder \n v1.1\n" (at 160.190782 82.392253) (layer "B.SilkS")
+    (effects (font (size 1 1) (thickness 0.25) bold) (justify mirror))
+  )
   (gr_text "Flipper Add-On\nMarauder \n v1.1\n" (at 174.07 86.12) (layer "F.SilkS")
     (effects (font (size 1 1) (thickness 0.25) bold))
