File: Marauder/Marauder.kicad_pcb (KiCad board)
At the start: 2 copper layers, 67 x 28 mm, 50 parts, among them J1 Conn_01x08_Socket, J2 Conn_01x08_Socket, J3 Conn_01x10_Socket, J4 GPS, J5 Conn_01x10_Socket, P1 USB_C_Plug_USB2.0, Q1 DMP2004TK-7, Q2 DMP2004TK-7, SW1 RESET, SW2 BOOT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

Commit message: feat: rename addons
Other:
- board text added: "Flipper Addon Marauder v1.1"
- board text removed: "Flipper Add-On Marauder v1.1"
