File: Marauder/Marauder.kicad_sch (KiCad schematic)
At the start: 23 parts, among them J1 Conn_01x08_Socket, J2 Conn_01x08_Socket, J3 Conn_01x10_Socket, J4 GPS, J5 Conn_01x10_Socket, P1 USB_C_Plug_USB2.0, Q1 DMP2004TK-7, Q2 DMP2004TK-7, SW1 RESET, SW2 GPIO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

Commit message: Routing finished of flipper marauder
Connections:
- no-connect marks 26 -> 27
Changed lines of the file:
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@@
   (no_connect (at 187.071 56.896))
   (no_connect (at 181.356 79.756))
+  (no_connect (at 227.711 67.056))
   (no_connect (at 227.711 56.896))
   (no_connect (at 181.356 82.296))

Commit message: BOM of flipper marauder generated
Parts:
- J2: LCSC# C2894950 -> (none); now not fitted
- J4: now not fitted
- J5: LCSC# C492418 -> (none); manf# PZ254R-11-10P -> (none); now not fitted
Other:
- moved on the sheet: J1

Commit message: BOM updated
Parts:
- J1: LCSC# C2894950 -> C492407; manf# PZ254-1-08-W-8.5 -> (none)
- J2: LCSC# (none) -> C492407
- J3: LCSC# C492418 -> C57369
- J5: LCSC# (none) -> C57369
- R3, R4: LCSC# C191782 -> C156350
- SW1, SW2: LCSC# C2886897 -> (none); manf# (none) -> TL3342F450QG
Changed lines of the file:
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@@
       (effects (font (size 1.27 1.27)) hide)
     )
-    (property "LCSC#" "C191782" (at 129.54 40.767 0)
+    (property "LCSC#" "C156350" (at 129.54 40.767 0)
       (effects (font (size 1.27 1.27)) hide)
     )
@@
       (effects (font (size 1.27 1.27)) hide)
     )
-    (property "LCSC#" "C492418" (at 32.6898 76.073 0)
+    (property "LCSC#" "C57369" (at 32.6898 76.073 0)
       (effects (font (size 1.27 1.27)) hide)
     )
@@
       (effects (font (size 1.27 1.27)) hide)
     )
-    (property "LCSC#" "" (at 55.118 76.073 0)
+    (property "LCSC#" "C57369" (at 55.118 76.073 0)
       (effects (font (size 1.27 1.27)) hide)
     )
@@
       (effects (font (size 1.27 1.27)) hide)
     )
-    (property "LCSC#" "C191782" (at 129.54 43.307 0)
+    (property "LCSC#" "C156350" (at 129.54 43.307 0)
       (effects (font (size 1.27 1.27)) hide)
     )
@@
       (effects (font (size 1.27 1.27)) hide)
     )
-    (property "manf#" "" (at 40.132 123.317 0)
-      (effects (font (size 1.27 1.27)) hide)
-    )
-    (property "LCSC#" "C2886897" (at 40.132 123.317 0)
+    (property "manf#" "TL3342F450QG" (at 40.132 123.317 0)
+      (effects (font (size 1.27 1.27)) hide)
+    )
+    (property "LCSC#" "" (at 40.132 123.317 0)
       (effects (font (size 1.27 1.27)) hide)
     )
@@
       (effects (font (size 1.27 1.27)) hide)
     )
-    (property "manf#" "PZ254-1-08-W-8.5" (at 32.512 37.973 0)
-      (effects (font (size 1.27 1.27)) hide)
-    )
-    (property "LCSC#" "C2894950" (at 32.512 37.973 0)
+    (property "manf#" "" (at 32.512 37.973 0)
+      (effects (font (size 1.27 1.27)) hide)
+    )
+    (property "LCSC#" "C492407" (at 32.512 37.973 0)
       (effects (font (size 1.27 1.27)) hide)
     )
@@
       (effects (font (size 1.27 1.27)) hide)
     )
-    (property "manf#" "" (at 42.037 142.621 0)
-      (effects (font (size 1.27 1.27)) hide)
-    )
-    (property "LCSC#" "C2886897" (at 42.037 142.621 0)
+    (property "manf#" "TL3342F450QG" (at 42.037 142.621 0)
+      (effects (font (size 1.27 1.27)) hide)
+    )
+    (property "LCSC#" "" (at 42.037 142.621 0)
       (effects (font (size 1.27 1.27)) hide)
     )
@@
       (effects (font (size 1.27 1.27)) hide)
     )
-    (property "LCSC#" "" (at 52.324 37.973 0)
-      (effects (font (size 1.27 1.27)) hide)
-    )
+    (property "LCSC#" "C492407" (at 52.324 37.973 0)
+      (effects (font (size 1.27 1.27)) hide)
+    )

Commit message: Marauder's BOM updated
Parts:
- U2: value ESP32-S3-WROOM-1U-N16 -> ESP32-S3-WROOM-1U-N4; manf# ESP32-S3-WROOM-1U-N16 -> ESP32-S3-WROOM-1U-N4
Changed lines of the file:
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@@
       (effects (font (size 1.524 1.524)))
     )
-    (property "Value" "ESP32-S3-WROOM-1U-N16" (at 207.391 28.956 0)
+    (property "Value" "ESP32-S3-WROOM-1U-N4" (at 207.391 28.956 0)
       (effects (font (size 1.524 1.524)))
     )
@@
       (effects (font (size 1.524 1.524)) hide)
     )
-    (property "manf#" "ESP32-S3-WROOM-1U-N16" (at 187.071 36.576 0)
+    (property "manf#" "ESP32-S3-WROOM-1U-N4" (at 187.071 36.576 0)
       (effects (font (size 1.27 1.27)) hide)
     )
