File: FLIPPER_MOD_BUS/FLIPPER_MOD_BUS.kicad_pcb (KiCad board)
At the start: 2 copper layers, 62.8 x 23.2 mm, 26 parts, among them J1 Conn_01x02, J2 Conn_01x10_Socket, J3 Conn_01x08_Socket, J4 Conn_01x02_Socket, U1 SP3485EN

Commit message: fix(hw): Differential Pair
Parts:
- added R8: 60, Resistor_SMD:R_1206_3216Metric_Pad1.30x1.75mm_HandSolder, F.Cu at (170.0, 92.6)
- R6: value 120 -> 60; footprint Resistor_SMD:R_0603_1608Metric_Pad0.98x0.95mm_HandSolder -> Resistor_SMD:R_1206_3216Metric_Pad1.30x1.75mm_HandSolder
- moved R7 5.63 mm to (166.5, 94.2), turned to 180 degrees
- moved R6 5.62 mm to (170.1, 81.3)
- moved R5 5.54 mm to (166.5, 79.8), turned to 0 degrees
- moved J4 2.74 mm to (170.1, 88.2)
Connections:
- J4 pad 1: /RS485A -> Net-(J4-Pin_1)
Routing:
- net /RS485A: track 15.0 -> 23.6 mm
- net /RS485B: track 14.8 -> 23.2 mm
- net Net-(J4-Pin_1): track 0.00 -> 2.83 mm
- net +3V3: track 68.4 -> 66.0 mm
Other:
- board text added: "FLIPPER SHIELD MODBUS V1.2"
- board text removed: "FLIPPER SHIELD MODBUS V1.1"

Commit message: fix: nets conflict solved & version label updated
Routing:
- net /DE: track 33.8 -> 37.2 mm
Other:
- board text added: "FLIPPER SHIELD MODBUS V1.3"
- board text removed: "FLIPPER SHIELD MODBUS V1.2"
Changed lines of the file:
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@@
 		(tags "resistor handsolder")
 		(property "Reference" "R5"
-			(at -2.811 -0.022 360)
+			(at -2.811 -0.022 0)
 			(layer "F.SilkS")
 			(effects
@@
 		)
 		(property "Value" "20K"
-			(at 0 1.43 360)
+			(at 0 1.43 0)
 			(layer "F.Fab")
 			(effects
@@
 		)
 		(fp_text user "${REFERENCE}"
-			(at 0 0 360)
+			(at 0 0 0)
 			(layer "F.Fab")
 			(effects
@@
 		)
 		(property "LCSC#" "C25586"
-			(at 0 0 270)
+			(at 0 0 -90)
 			(layer "F.Fab")
 			(hide yes)
@@
 		)
 		(property "Proveedor" "LCSC"
-			(at 0 0 270)
+			(at 0 0 -90)
 			(layer "F.Fab")
 			(hide yes)
@@
 		)
 		(property "manf#" "0603WAJ0203T5E"
-			(at 0 0 270)
+			(at 0 0 -90)
 			(layer "F.Fab")
 			(hide yes)
@@
 		(layer "Edge.Cuts")
 	)
-	(gr_text "FLIPPER SHIELD\nMODBUS V1.2"
+	(gr_text "FLIPPER SHIELD\nMODBUS V1.3"
 		(at 150 90 0)
 		(layer "B.SilkS")
@@
 		)
 	)
-	(gr_text "FLIPPER SHIELD\nMODBUS V1.2\n"
+	(gr_text "FLIPPER SHIELD\nMODBUS V1.3\n"
 		(at 129.995 91.63 0)
 		(layer "F.SilkS")
@@
 		(net 1)
 	)
-	(segment
-		(start 161.338 98.5)
-		(end 161.338 96.942)
-		(width 0.5)
-		(layer "F.Cu")
-		(net 1)
-	)
 	(via
 		(at 164.4904 89.8906)
@@
 	)
 	(segment
+		(start 161.338 98.5)
+		(end 161.338 96.942)
+		(width 0.5)
+		(layer "B.Cu")
+		(net 1)
+	)
+	(segment
 		(start 162.9156 85.471)
 		(end 162.9156 93.3356)
@@
 	)
 	(segment
-		(start 162.4 87.61)
-		(end 162.77 87.24)
+		(start 162.77 87.41)
+		(end 162.77 84.04)
 		(width 0.25)
 		(layer "B.Cu")
@@
 	)
 	(segment
-		(start 162.77 87.24)
-		(end 162.77 85.68)
+		(start 171.498 84.008)
+		(end 171.498 98.5)
 		(width 0.25)
 		(layer "B.Cu")
@@
 	)
 	(segment
-		(start 163.09 85.36)
-		(end 171.15 85.36)
+		(start 162.57 87.61)
+		(end 162.77 87.41)
 		(width 0.25)
 		(layer "B.Cu")
@@
 	)
 	(segment
-		(start 157.2568 87.61)
-		(end 162.4 87.61)
+		(start 157.2514 87.6046)
+		(end 157.2568 87.61)
 		(width 0.25)
 		(layer "B.Cu")
@@
 	)
 	(segment
-		(start 171.498 85.708)
-		(end 171.498 98.5)
+		(start 163.07 83.74)
+		(end 171.23 83.74)
 		(width 0.25)
 		(layer "B.Cu")
@@
 	)
 	(segment
-		(start 171.15 85.36)
-		(end 171.498 85.708)
+		(start 157.2568 87.61)
+		(end 162.57 87.61)
 		(width 0.25)
 		(layer "B.Cu")
@@
 	)
 	(segment
-		(start 157.2514 87.6046)
-		(end 157.2568 87.61)
+		(start 162.77 84.04)
+		(end 163.07 83.74)
 		(width 0.25)
 		(layer "B.Cu")
@@
 	)
 	(segment
-		(start 162.77 85.68)
-		(end 163.09 85.36)
+		(start 171.23 83.74)
+		(end 171.498 84.008)
 		(width 0.25)
 		(layer "B.Cu")
