File: FLIPPER_MAGSPOOF/mags.kicad_sch (KiCad schematic)
At the start: 10 parts, among them J1 Coil, J2 Conn_01x10_Socket, J3 Conn_01x08_Socket, J4 Conn_01x08_Socket, J5 Conn_01x10_Socket, J6 Coil, SW1 On, U3 TC4424

Commit message: feat(hw): change SW1 part and footprint
Parts:
- SW1: footprint footprintsg:JS102011SAQN -> Library:MSK12C02; LCSC# C221660 -> C431540; manf# JS102011SAQN -> MSK12C02
Changed lines of the file:
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@@
 			)
 		)
-		(property "Footprint" "footprintsg:JS102011SAQN"
+		(property "Footprint" "Library:MSK12C02"
 			(at 63.5 63.5 0)
 			(effects
@@
 			)
 		)
-		(property "LCSC#" "C221660"
+		(property "LCSC#" "C431540"
 			(at 63.5 63.5 0)
 			(effects
@@
 			)
 		)
-		(property "manf#" "JS102011SAQN"
+		(property "manf#" "MSK12C02"
 			(at 63.5 63.5 0)
 			(effects
