File: FLIPPER_ETHERNET/FLIPPER_ETHERNET.kicad_pcb (KiCad board)
At the start: 2 copper layers, 67 x 25 mm, 38 parts, among them J1 RJ45_Hanrun_HR911105A_Horizon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, J2 Conn_01x08_Socket, J3 Conn_01x10_Socket, U1 ENC28J60x-SO, Y1 25MHz

Commit message: feat(hw): Update labels
Parts:
- added G***: LOGO, CatSniffer:calderon, B.Cu at (151.2, 56.0)
Routing:
- net /LEDB: track 62.0 -> 58.9 mm
- net /LEDA: track 78.2 -> 76.2 mm
Other:
- board text added: "FLIPPER ADDON ETHERNET v1.1"
- board text removed: "FLIPPER ADDON ETHERNET v1.0"
