File: FLIPPER_CANBUS/CANBUS_Flipper.kicad_pcb (KiCad board)
At the start: 2 copper layers, 67 x 21.3 mm, 42 parts, among them J1 Conn_01x08_Socket, J2 Conn_01x10_Socket, J3 Conn, U3 MCP251863T-H-SS, Y1 40MHz

Commit message: feat(Hw):Update_Schematic
Connections:
- net /CLK renamed /CLKO
Changed lines of the file:
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@@
 	(net 32 "unconnected-(U3-NC-Pad27)")
 	(net 33 "unconnected-(U3-NC-Pad12)")
-	(net 34 "/CLK")
+	(net 34 "/CLKO")
 	(footprint "Aesthetics:electronic_cats_logo_8x6"
 		(layer "F.Cu")
@@
 			(layers "*.Cu" "*.Mask")
 			(remove_unused_layers no)
-			(net 34 "/CLK")
+			(net 34 "/CLKO")
 			(pinfunction "Pin_3")
 			(pintype "passive")
@@
 			(size 1 1.5)
 			(layers "F.Cu" "F.Mask")
-			(net 34 "/CLK")
+			(net 34 "/CLKO")
 			(pinfunction "A")
 			(pintype "passive")
